File: LPF_Butterworth_Filter.kicad_sch (KiCad schematic)
At the start: 0 parts

Commit message: sma footprints added
Parts:
- added U1, U2: (no value), Filter_Lib:CONN SMA RCPT STR 50OHM EDGE MNT, symbol Filter_Materials:CONN_SMA_RCPT_STR_50OHM_EDGE_MNT
Connections:
- new net: U1.3 (Signal), U2.3 (Signal)
- new net GND: U1.5 (Ground), U2.5 (Ground)
